Commit message: fixes

File: geometry/franka/panda_arm_finger_long.urdf (robot description, URDF)
Before this commit: robot panda, 14 links, 13 joints
Links:
- link panda_leftfinger_lower: geometry collision mesh filename=meshes/collision/franka_finger_lower_long.stl; visual mesh filename=meshes/collision/franka_finger_lower_long.stl
- link panda_rightfinger_lower: geometry collision mesh filename=meshes/collision/franka_finger_lower_long.stl; visual mesh filename=meshes/collision/franka_finger_lower_long.stl

File: geometry/franka/panda_arm_finger_orig.urdf (robot description, URDF)
Before this commit: robot panda, 14 links, 13 joints
Links:
- link panda_leftfinger_lower: geometry collision mesh filename=meshes/collision/franka_finger_lower_orig.stl; visual mesh filename=meshes/collision/franka_finger_lower_orig.stl
- link panda_rightfinger_lower: geometry collision mesh filename=meshes/collision/franka_finger_lower_orig.stl; visual mesh filename=meshes/collision/franka_finger_lower_orig.stl
