Commit message: fix hand_joint from revolute

File: data/franka/panda_arm_finger_long.urdf (robot description, URDF)
Before this commit: robot panda, 14 links, 13 joints
Joints:
- joint panda_hand_joint: axis 0 0 1 -> (none); limit lower=-0.78 upper=-0.78 effort=12 velocity=0.01 -> (none); origin xyz=0 0 0 rpy=0 0 0 -> xyz=0 0 0 rpy=0 0 -0.785; type revolute -> fixed

File: data/franka/panda_arm_finger_orig.urdf (robot description, URDF)
Before this commit: robot panda, 14 links, 13 joints
Joints:
- joint panda_hand_joint: axis 0 0 1 -> (none); limit lower=-0.78 upper=-0.78 effort=12 velocity=0.01 -> (none); origin xyz=0 0 0 rpy=0 0 0 -> xyz=0 0 0 rpy=0 0 -0.785; type revolute -> fixed

File: data/franka/panda_arm_finger_wide_curved.urdf (robot description, URDF)
Before this commit: robot panda, 14 links, 13 joints
Joints:
- joint panda_hand_joint: axis 0 0 1 -> (none); limit lower=-0.78 upper=-0.78 effort=12 velocity=0.01 -> (none); origin xyz=0 0 0 rpy=0 0 0 -> xyz=0 0 0 rpy=0 0 -0.785; type revolute -> fixed

File: data/franka/panda_arm_finger_wide_flat.urdf (robot description, URDF)
Before this commit: robot panda, 14 links, 13 joints
Joints:
- joint panda_hand_joint: axis 0 0 1 -> (none); limit lower=-0.78 upper=-0.78 effort=12 velocity=0.01 -> (none); origin xyz=0 0 0 rpy=0 0 0 -> xyz=0 0 0 rpy=0 0 -0.785; type revolute -> fixed
