Commit message: sync tri

File: data/peg/peg.urdf (robot description, URDF)
Before this commit: robot peg.urdf, 1 links, 0 joints
Links:
- link baseLink: mass 0.1 -> 0.5

File: data/peg_block/peg_block.urdf (robot description, URDF)
Before this commit: robot peg_block.urdf, 1 links, 0 joints
Links:
- link baseLink: geometry collision mesh filename=peg_block_small.obj scale=2 1.5 1.5; visual mesh filename=peg_block_small.obj scale=2 1.5 1.5
